File: pipe_v1.kicad_pcb (KiCad board)
At the start: 2 copper layers, 27.9 x 22.9 mm, 8 parts, among them Q1 BC548, Q2 BC558

Commit message: Refactoring on PCB design
Parts:
- Q1, Q2: footprint Pipe:TO-92 -> Package_TO_SOT_THT:TO-92_Inline
Routing:
- net Net-(C1-Pad1): track 9.68 -> 12.2 mm
- net Net-(C1-Pad2): track 22.9 -> 24.4 mm
- net Net-(Q1-Pad1): track 5.50 -> 6.13 mm
- net Net-(D1-Pad1): track 5.45 -> 6.09 mm
